File: DroneProject/DroneProject.kicad_sch (KiCad schematic)
At the start: 4 parts, among them U1 DRV8210PDSGR, U2 ESP32-WROOM-32E 4MB

Commit message: Worked on the schematics
Parts:
- added C3, C4, C5: C, symbol Device:C
- added R1, R2: 10K, symbol Device:R_US
- added U3: BMI323, BMI323_BOS, symbol 2025-09-30_23-20-55:BMI323
Connections:
- net BATT: now also C1.2; no longer C1.1, C2.2, U1.8 (VCC)
- net GND: now also C1.1, U1.4 (GND), U1.9 (Thermal_Pad), U2.1 (GND), C3.2, C4.2, C5.2, U3.6 (GNDIO), U3.7 (GND); no longer C1.2
- net IN2BMI: now reaches U2.10 (IO25)
- net 3V3: now reaches U2.2 (3V3)
- net 3V3: now also C2.2, U1.8 (VCC), C3.1, C4.1, R1.1, R2.1, U3.8 (VDD)
- net at U2.3 (EN): now also R1.2
- net at U2.38 (GND): now also U2.39 (GND), U2.40 (GND), U2.41 (GND), U2.42 (GND), U2.43 (GND), U2.44 (GND), U2.45 (GND), U2.46 (GND), U2.47 (GND), C5.1
- net IN1DRV: now reaches U2.6 (IO34)
- net IN1BMI: now reaches U2.7 (IO35)
- net IN2DRV: now reaches U2.8 (IO32)
- net VDDI0: now reaches U2.9 (IO33)
- net MOTOR: now reaches U1.2 (OUT1)
- net MOTOR: now also U1.3 (OUT2)
- net IO32: now reaches U1.5 (IN2)
- net IO34: now reaches U1.6 (IN1)
- net at U1.7 (SLEEP_N): now also R2.2
- new net FLASHMEM: U3.1 (SDO)
- new net IO25: U3.9 (INT2)
- new net IO33: U3.12 (CSB), U3.5 (VDDIO)
- new net IO35: U3.4 (INT1)
- no-connect marks 1 -> 3
Other:
- note added: "Christ-Ismael Kone: My First Drone >:D"
- moved on the sheet: U1, U2
